File: TH_SMD_Kit/blinky_kit_pcb/blinky_kit_pcb.kicad_pcb (KiCad board)
At the start: 2 copper layers, 38.1 x 38.1 mm, 13 parts, among them J1 1-0000120, Q1 1-0000036, Q2 1-0000036

Commit message: Add made by line
Other:
- board text added: "+"
- board text added: "-"
- board text added: "3-0000080"
- board text added: "Leeman Geophysical LLC"
- board text added: "Made By"
