File: TH_SMD_Kit/blinky_kit_pcb/blinky_kit_pcb.sch (KiCad schematic (older format))
At the start: 12 parts, among them J1 1-0000120, Q1 1-0000036, Q2 1-0000036

Commit message: Fix schematic
Other:
- moved on the sheet: Q1
Changed lines of the file:
@@
 L transistors:1-0000036 Q1
 U 1 1 6077AAAC
-P 4600 4350
-F 0 "Q1" H 4791 4396 50  0000 L CNN
-F 1 "1-0000036" H 4800 4300 50  0001 L CNN
-F 2 "transistors:1-0000036" H 4800 4450 50  0001 C CNN
-F 3 "~" H 4600 4350 50  0001 C CNN
-F 4 "1-0000036" H 4600 4350 50  0001 C CNN "Internal Part Number"
-F 5 "1" H 4600 4350 50  0001 C CNN "Populated"
-F 6 "MMBT3904" H 4791 4305 50  0000 L CNN "PValue"
-	1    4600 4350
-	1    0    0    -1
+P 4800 4350
+F 0 "Q1" H 4991 4396 50  0000 L CNN
+F 1 "1-0000036" H 5000 4300 50  0001 L CNN
+F 2 "transistors:1-0000036" H 5000 4450 50  0001 C CNN
+F 3 "~" H 4800 4350 50  0001 C CNN
+F 4 "1-0000036" H 4800 4350 50  0001 C CNN "Internal Part Number"
+F 5 "1" H 4800 4350 50  0001 C CNN "Populated"
+F 6 "MMBT3904" H 4991 4305 50  0000 L CNN "PValue"
+	1    4800 4350
+	-1   0    0    -1
 $EndComp
 $Comp
@@
 	-1   0    0    1
 $EndComp
-Wire Wire Line
-	5900 3750 5900 4075
-Wire Wire Line
-	5900 4075 4400 4075
-Wire Wire Line
-	4400 4075 4400 4350
 Connection ~ 5900 3750
+Wire Wire Line
+	5900 4350 5000 4350
+Wire Wire Line
+	5900 3750 5900 4350
 $EndSCHEMATC

Commit message: Changed NP connector
Parts:
- removed J1: 1-0000120, Connector_Wire:SolderWire-0.5sqmm_1x02_P4.6mm_D0.9mm_OD2.1mm_Relief, symbol connectors:1-0000120
- added J?: NP_Conn_01x02, np_connectors:PinHeader_1x02_P2.54mm_Vertical, symbol np_connectors:NP_Conn_01x02
- C1, C2: symbol capacitors_th:1-0000853 -> blinky_kit_pcb-rescue:1-0000853-capacitors_th
- D1, D2: symbol leds_th:1-0000568 -> blinky_kit_pcb-rescue:1-0000568-leds_th
Connections:
- net GND: now also J?.1 (Pin_1)
- net VCC: now also J?.2 (Pin_2)
Changed lines of the file:
@@
 $EndComp
 $Comp
-L capacitors_th:1-0000853 C2
+L blinky_kit_pcb-rescue:1-0000853-capacitors_th C2
 U 1 1 60773993
 P 6350 3750
@@
 $EndComp
 $Comp
-L capacitors_th:1-0000853 C1
+L blinky_kit_pcb-rescue:1-0000853-capacitors_th C1
 U 1 1 60774DDD
 P 5050 3750
@@
 $EndComp
 $Comp
-L leds_th:1-0000568 D2
+L blinky_kit_pcb-rescue:1-0000568-leds_th D2
 U 1 1 6077414F
 P 6700 2750
@@
 $EndComp
 $Comp
-L leds_th:1-0000568 D1
+L blinky_kit_pcb-rescue:1-0000568-leds_th D1
 U 1 1 60774DCC
 P 4700 2750
@@
 Wire Wire Line
 	1300 2150 1300 2300
-$Comp
-L connectors:1-0000120 J1
-U 1 1 607A99AA
+Connection ~ 5900 3750
+Wire Wire Line
+	5900 4350 5000 4350
+Wire Wire Line
+	5900 3750 5900 4350
+$Comp
+L np_connectors:NP_Conn_01x02 J?
+U 1 1 608062AB
 P 1000 2150
-F 0 "J1" H 918 1825 50  0000 C CNN
-F 1 "1-0000120" H 1000 1950 50  0001 C CNN
-F 2 "Connector_Wire:SolderWire-0.5sqmm_1x02_P4.6mm_D0.9mm_OD2.1mm_Relief" H 1000 2150 50  0001 C CNN
+F 0 "J?" H 1000 1950 50  0000 C CNN
+F 1 "NP_Conn_01x02" H 1000 1950 50  0001 C CNN
+F 2 "np_connectors:PinHeader_1x02_P2.54mm_Vertical" H 1000 2150 50  0001 C CNN
 F 3 "~" H 1000 2150 50  0001 C CNN
-F 4 "1-0000120" H 1000 2150 50  0001 C CNN "Internal Part Number"
-F 5 "1" H 1000 2150 50  0001 C CNN "Populated"
-F 6 "TSW-102-07-T-S" H 918 1916 50  0000 C CNN "PValue"
+F 4 "0-0000000" H 1000 2150 50  0001 C CNN "Internal Part Number"
+F 5 "0" H 1000 2150 50  0001 C CNN "Populated"
+F 6 "NP_Conn_01x02" H 1025 2250 50  0000 C CNN "PValue"
 	1    1000 2150
 	-1   0    0    1
 $EndComp
-Connection ~ 5900 3750
-Wire Wire Line
-	5900 4350 5000 4350
-Wire Wire Line
-	5900 3750 5900 4350
 $EndSCHEMATC
