File: TH_SMD_Kit/KiCAD_Project/blinky_kit_pcb/blinky_kit_pcb.kicad_pcb (KiCad board)
At the start: 2 copper layers, 38.1 x 38.1 mm, 13 parts, among them J1 1-0000120, Q1 1-0000036, Q2 1-0000036

Commit message: TH and SMD Rev 1.0 Production
Parts:
- added PCB1: barepcb, misc:barepcb, F.Cu at (276.1, 160.5)
- J1: value 1-0000120 -> 2 Pos
Routing:
- net GND: track 1.69 -> 3.96 mm, vias 1 -> 2
Other:
- board text added: "+"
- board text added: "-"
- board text added: "3-0000080"
- board text added: "Leeman Geophysical LLC"
- board text added: "Made By"
